Commit message: Rebase from 'upstream'

File: gz_ros2_control_demos/urdf/test_ackermann_drive.xacro.urdf (robot description, URDF)
Before this commit: robot ackermann_drive, 8 links, 7 joints
Joints:
- joint front_left_wheel_joint: origin xyz=0 0 0 rpy=0 0 0 -> xyz=0 0 0 rpy=-1.57 0 0
- joint front_right_wheel_joint: origin xyz=0 0 0 rpy=0 0 0 -> xyz=0 0 0 rpy=-1.57 0 0
- joint left_wheel_steering_joint: axis 0 1 0 -> 0 0 1; origin xyz=0.9 -0.5 -0.2 rpy=1.57 0 0 -> xyz=0.9 0.5 -0.2 rpy=0 0 0
- joint right_wheel_steering_joint: axis 0 1 0 -> 0 0 1; origin xyz=0.9 0.5 -0.2 rpy=1.57 0 0 -> xyz=0.9 -0.5 -0.2 rpy=0 0 0
