Commit message: Imported upstream version '0.7.14' of 'upstream'

File: gz_ros2_control_demos/urdf/test_cart_position.xacro.urdf (robot description, URDF)
Before this commit: robot cartopole, 3 links, 2 joints
Links:
- link cart: geometry visual box size=0.5 0.5 0.2
- link slideBar: geometry visual box size=30 0.05 0.05

File: gz_ros2_control_demos/urdf/test_cart_velocity.xacro.urdf (robot description, URDF)
Before this commit: robot cartopole, 6 links, 5 joints
Links:
- removed link world
Joints:
- removed joint world_to_base

File: gz_ros2_control_demos/urdf/test_gripper_mimic_joint.xacro.urdf (robot description, URDF)
Before this commit: robot gripper, 4 links, 3 joints
Links:
- link base: geometry visual box size=0.5 1 1
- link finger_left: mass 4 -> 5
- link finger_right: mass 4 -> 5

Commit message: Imported upstream version '1.2.13' of 'upstream'

File: gz_ros2_control_demos/urdf/test_cart_position.xacro.urdf (robot description, URDF)
Before this commit: robot cartopole, 3 links, 2 joints
Links:
- link cart: geometry collision box size=0.5 0.5 0.2; visual box size=0.5 0.5 0.2
- link slideBar: geometry collision box size=30 0.05 0.05; visual box size=30 0.05 0.05

File: gz_ros2_control_demos/urdf/test_cart_velocity.xacro.urdf (robot description, URDF)
Before this commit: robot cartopole, 5 links, 4 joints
Links:
- added link world
Joints:
- added joint world_to_base: type fixed, parent world, child slideBar, origin xyz=0 0 1 rpy=0 0 0

File: gz_ros2_control_demos/urdf/test_gripper_mimic_joint_effort.xacro.urdf (robot description, URDF)
Before this commit: robot gripper, 4 links, 3 joints
Links:
- link base: geometry collision box size=0.5 1 1; visual box size=0.5 1 1
- link finger_left: mass 5 -> 4
- link finger_right: mass 5 -> 4

Commit message: Imported upstream version '0.7.20' of 'upstream'

File: gz_ros2_control_demos/urdf/test_cart_position.xacro.urdf (robot description, URDF)
Before this commit: robot cartopole, 3 links, 2 joints
Links:
- link cart: geometry visual box size=0.5 0.5 0.2
- link slideBar: geometry visual box size=30 0.05 0.05

File: gz_ros2_control_demos/urdf/test_cart_velocity.xacro.urdf (robot description, URDF)
Before this commit: robot cartopole, 6 links, 5 joints
Links:
- removed link world
Joints:
- removed joint world_to_base
