Commit message: Imported upstream version '4.0.1' of 'upstream'

File: gz_ros2_control_demos/urdf/test_cart_position.xacro.urdf (robot description, URDF)
Before this commit: robot cartopole, 3 links, 2 joints
Links:
- link cart: geometry collision box size=0.5 0.5 0.2; visual box size=0.5 0.5 0.2
- link slideBar: geometry collision box size=30 0.05 0.05; visual box size=30 0.05 0.05

File: gz_ros2_control_demos/urdf/test_cart_velocity.xacro.urdf (robot description, URDF)
Before this commit: robot cartopole, 5 links, 4 joints
Links:
- added link world
Joints:
- added joint world_to_base: type fixed, parent world, child slideBar, origin xyz=0 0 1 rpy=0 0 0
