Commit message: Imported upstream version '0.7.21' of 'upstream'

File: gz_ros2_control_demos/urdf/test_gripper_mimic_joint_position.xacro.urdf (robot description, URDF)
Before this commit: robot gripper, 4 links, 3 joints
Joints:
- joint left_finger_joint: mimic joint=right_finger_joint multiplier=1.0 offset=0.05 -> joint=right_finger_joint
